File: mm_external_uart.kicad_sch (KiCad schematic)
At the start: 0 parts

Commit message: tp2
Parts:
- added C7: 0.1uF 16V, symbol Device:C_Small
- added C7: 2.2uF 16V, symbol Device:C_Small
- added J2: Conn_01x04, symbol Connector_Generic:Conn_01x04
- added R8: 100, Resistor_SMD:R_0603_1608Metric, symbol Device:R
Connections:
- new net: J2.3 (Pin_3), R8.2
- new net +3.3V: C7.1, C7.1, J2.1 (Pin_1)
- new net EXT_UART_RX: J2.4 (Pin_4)
- new net EXT_UART_TX: R8.1
- new net GND: C7.2, C7.2, J2.2 (Pin_2)

Commit message: updated to kicad 8.0
Parts:
- renumbered C7 to C10, C7 to C19, R8 to R19
