File: mm_mcu.kicad_sch (KiCad schematic)
At the start: 18 parts, among them J1 Conn_ARM_JTAG_SWD_10, U1 STM32F030C8Tx

Commit message: tp2
Other:
- moved on the sheet: BOOT0, C1, C2, C3, C4, C5, C6, R1, R2, R3, R4, R5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
