File: mm_power.kicad_sch (KiCad schematic)
At the start: 1 part, among them J5 Conn_01x02

Commit message: tp2
Parts:
- added C7: 22uF, symbol Device:C_Small
- added C8: 1uF, symbol Device:C_Small
- added D1: GREEN, symbol Device:LED_Small
- added R12: 680R, symbol Device:R_Small
- added U2: LP5907MFX-3.3, Package_TO_SOT_SMD:SOT-23-5, symbol Regulator_Linear:LP5907MFX-3.3
Connections:
- net +BATT: now also C7.1, U2.1 (IN), U2.3 (EN)
- net GND: now also C7.2, C8.2, D1.1 (K), U2.2 (GND)
- new net: D1.2 (A), R12.2
- new net +3.3V: C8.1, R12.1, U2.5 (OUT)
